Commit message: Update CRX-10iA_L.urdf with joint limits & velocities

File: CRX-10iA_L/urdf/CRX-10iA_L.urdf (robot description, URDF)
Before this commit: robot CRX-10iA_L, 7 links, 6 joints
Joints:
- joint Joint_1: limit lower=0 upper=0 effort=0 velocity=0 -> lower=0 upper=6.632251 effort=0 velocity=2.094395
- joint Joint_2: limit lower=0 upper=0 effort=0 velocity=0 -> lower=0 upper=6.283185 effort=0 velocity=2.094395
- joint Joint_3: limit lower=0 upper=0 effort=0 velocity=0 -> lower=0 upper=9.948377 effort=0 velocity=3.141593
- joint Joint_4: limit lower=0 upper=0 effort=0 velocity=0 -> lower=0 upper=6.6323 effort=0 velocity=3.1416
- joint Joint_5: limit lower=0 upper=0 effort=0 velocity=0 -> lower=0 upper=6.2832 effort=0 velocity=3.1416
- joint Joint_6: axis -1 0 0 -> 0 0 0; limit (none) -> lower=0 upper=7.854 effort=0 velocity=3.1416; type fixed -> revolute
