Commit message: compile error: fixes to package.xml

File: src/fanuc/urdf/fanuc.urdf (robot description, URDF)
Before this commit: robot CRX-10iA_L, 8 links, 7 joints
Links:
- link Link_1: geometry collision mesh filename=package://fanuc/meshes/Link_1.STL; visual mesh filename=package://fanuc/meshes/Link_1.STL
- link Link_2: geometry collision mesh filename=package://fanuc/meshes/Link_2.STL; visual mesh filename=package://fanuc/meshes/Link_2.STL
- link Link_3: geometry collision mesh filename=package://fanuc/meshes/Link_3.STL; visual mesh filename=package://fanuc/meshes/Link_3.STL
- link Link_4: geometry collision mesh filename=package://fanuc/meshes/Link_4.STL; visual mesh filename=package://fanuc/meshes/Link_4.STL
- link Link_5: geometry collision mesh filename=package://fanuc/meshes/Link_5.STL; visual mesh filename=package://fanuc/meshes/Link_5.STL
- link Link_6: geometry collision mesh filename=package://fanuc/meshes/Link_6.STL; visual mesh filename=package://fanuc/meshes/Link_6.STL
- link base_link: geometry collision mesh filename=package://fanuc/meshes/base_link.STL; visual mesh filename=package://fanuc/meshes/base_link.STL

Commit message: Corrected orientation of robot

File: src/fanuc/urdf/fanuc.urdf (robot description, URDF)
Before this commit: robot fanuc, 8 links, 7 joints
Joints:
- joint base_joint: origin xyz=0 0 0 rpy=0 0 0 -> xyz=0 0 0.0 rpy=-1.57 0 0

Commit message: inertias/masses also updated in original urdf

File: src/fanuc/urdf/fanuc.urdf (robot description, URDF)
Before this commit: robot fanuc, 8 links, 7 joints
Links:
- link Link_1: mass 40 -> 3.84000000
- link Link_2: mass 40 -> 11.52000000
- link Link_3: mass 40 -> 2.88000000
- link Link_4: mass 40 -> 8.64000000
- link Link_5: mass 40 -> 1.60000000
- link Link_6: mass 40 -> 1.60000000
- link base_link: mass 40 -> 9.92000000
Joints:
- joint Joint_1: limit lower=0 upper=6.632251 effort=0 velocity=2.094395 -> lower=-3.31613 upper=3.31613 effort=0 velocity=2.094395
- joint Joint_2: limit lower=0 upper=6.283185 effort=0 velocity=2.094395 -> lower=-3.14159 upper=3.14159 effort=0 velocity=2.094395
- joint Joint_3: limit lower=0 upper=9.948377 effort=0 velocity=3.141593 -> lower=-4.97419 upper=4.97419 effort=0 velocity=3.141593
- joint Joint_4: limit lower=0 upper=6.6323 effort=0 velocity=3.1416 -> lower=-3.31615 upper=3.31615 effort=0 velocity=3.1416
- joint Joint_5: limit lower=0 upper=6.2832 effort=0 velocity=3.1416 -> lower=-3.14159 upper=3.14159 effort=0 velocity=3.1416
- joint Joint_6: axis 0 0 0 -> 1 0 0; limit lower=0 upper=7.854 effort=0 velocity=3.1416 -> lower=-3.927 upper=3.927 effort=0 velocity=3.1416

Commit message: joint effort values added

File: src/fanuc/urdf/fanuc.urdf (robot description, URDF)
Before this commit: robot fanuc, 8 links, 7 joints
Joints:
- joint Joint_1: limit lower=-3.31613 upper=3.31613 effort=0 velocity=2.094395 -> lower=-3.31613 upper=3.31613 effort=50 velocity=2.094395
- joint Joint_2: limit lower=-3.14159 upper=3.14159 effort=0 velocity=2.094395 -> lower=-3.14159 upper=3.14159 effort=45 velocity=2.094395
- joint Joint_3: limit lower=-4.97419 upper=4.97419 effort=0 velocity=3.141593 -> lower=-4.97419 upper=4.97419 effort=40 velocity=3.141593
- joint Joint_4: limit lower=-3.31615 upper=3.31615 effort=0 velocity=3.1416 -> lower=-3.31615 upper=3.31615 effort=34.8 velocity=3.1416
- joint Joint_5: limit lower=-3.14159 upper=3.14159 effort=0 velocity=3.1416 -> lower=-3.14159 upper=3.14159 effort=26 velocity=3.1416
- joint Joint_6: limit lower=-3.927 upper=3.927 effort=0 velocity=3.1416 -> lower=-3.927 upper=3.927 effort=11 velocity=3.1416

File: src/fanuc/urdf/fanuc_gripper.urdf (robot description, URDF)
Before this commit: robot fanuc, 18 links, 17 joints
Joints:
- joint Joint_1: limit lower=-3.31613 upper=3.31613 effort=0 velocity=2.094395 -> lower=-3.31613 upper=3.31613 effort=50 velocity=2.094395
- joint Joint_2: limit lower=-3.14159 upper=3.14159 effort=0 velocity=2.094395 -> lower=-3.14159 upper=3.14159 effort=45 velocity=2.094395
- joint Joint_3: limit lower=-4.97419 upper=4.97419 effort=0 velocity=3.141593 -> lower=-4.97419 upper=4.97419 effort=40 velocity=3.141593
- joint Joint_4: limit lower=-3.31615 upper=3.31615 effort=0 velocity=3.1416 -> lower=-3.31615 upper=3.31615 effort=34.8 velocity=3.1416
- joint Joint_5: limit lower=-3.14159 upper=3.14159 effort=0 velocity=3.1416 -> lower=-3.14159 upper=3.14159 effort=26 velocity=3.1416
- joint Joint_6: limit lower=-3.927 upper=3.927 effort=0 velocity=3.1416 -> lower=-3.927 upper=3.927 effort=11 velocity=3.1416
