Commit message: robotiq140 gripper added to fanuc urdf model (new urdf created)

File: src/fanuc/urdf/fanuc_gripper.urdf (robot description, URDF)
Before this commit: robot fanuc, 8 links, 7 joints
Links:
- added link ee_link
- added link robotiq_140_base_link, mass 0.636951; collision mesh filename=package://fanuc/meshes/robotiq_140/collision/robotiq_140_ba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; visual mesh filename=package://fanuc/meshes/robotiq_140/visual/robotiq_140_base_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
- added link robotiq_140_left_finger_link, mass 0.027309; collision mesh filename=package://fanuc/meshes/robotiq_140/collision/robotiq_140_fi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; visual mesh filename=package://fanuc/meshes/robotiq_140/visual/robotiq_140_finge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
- added link robotiq_140_left_finger_tip_link, mass 0.019555; collision mesh filename=package://fanuc/meshes/robotiq_140/collision/robotiq_140_fi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; visual mesh filename=package://fanuc/meshes/robotiq_140/visual/robotiq_140_finge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
- added link robotiq_140_left_inner_knuckle_link, mass 0.029951; collision mesh filename=package://fanuc/meshes/robotiq_140/collision/robotiq_140_in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; visual mesh filename=package://fanuc/meshes/robotiq_140/visual/robotiq_140_inner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
- added link robotiq_140_left_knuckle_link, mass 0.018491; collision mesh filename=package://fanuc/meshes/robotiq_140/collision/robotiq_140_kn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; visual mesh filename=package://fanuc/meshes/robotiq_140/visual/robotiq_140_knuck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
- added link robotiq_140_right_finger_link, mass 0.027309; collision mesh filename=package://fanuc/meshes/robotiq_140/collision/robotiq_140_fi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; visual mesh filename=package://fanuc/meshes/robotiq_140/visual/robotiq_140_finge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
- added link robotiq_140_right_finger_tip_link, mass 0.019555; collision mesh filename=package://fanuc/meshes/robotiq_140/collision/robotiq_140_fi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; visual mesh filename=package://fanuc/meshes/robotiq_140/visual/robotiq_140_finge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
- added link robotiq_140_right_inner_knuckle_link, mass 0.029951; collision mesh filename=package://fanuc/meshes/robotiq_140/collision/robotiq_140_in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; visual mesh filename=package://fanuc/meshes/robotiq_140/visual/robotiq_140_inner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
- added link robotiq_140_right_knuckle_link, mass 0.018491; collision mesh filename=package://fanuc/meshes/robotiq_140/collision/robotiq_140_kn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; visual mesh filename=package://fanuc/meshes/robotiq_140/visual/robotiq_140_knuck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
Joints:
- added joint ee_fixed_joint: type fixed, parent Link_6, child ee_link, origin xyz=0.0 0.0 0.0 rpy=0.0 0.0 0
- added joint robotiq_140_base_joint: type fixed, parent ee_link, child robotiq_140_base_link, origin xyz=0.0 0.0 0.0 rpy=0.0 0.0 0.0
- added joint robotiq_140_left_finger_joint: type fixed, parent robotiq_140_left_knuckle_link, child robotiq_140_left_finger_link, origin xyz=0.00795779 -0.03073656 0.0 rpy=0 0 0
- added joint robotiq_140_left_finger_tip_joint: type continuous, parent robotiq_140_left_inner_knuckle_link, child robotiq_140_left_finger_tip_link, origin xyz=0.09441861 -0.03294127 0.0 rpy=0.0 0.0 0.0, axis 0 0 1, limit lower=-3.14 upper=3.14 effort=0.1 velocity=100.0, mimic joint=robotiq_140_left_knuckle_joint multiplier=-1
- added joint robotiq_140_left_inner_knuckle_joint: type continuous, parent robotiq_140_base_link, child robotiq_140_left_inner_knuckle_link, origin xyz=0.06142 0.0127 0 rpy=3.14 0.0 0.0, axis 0 0 1, limit lower=-3.14 upper=3.14 effort=0.1 velocity=100.0, mimic joint=robotiq_140_left_knuckle_joint offset=0
- added joint robotiq_140_left_knuckle_joint: type revolute, parent robotiq_140_base_link, child robotiq_140_left_knuckle_link, origin xyz=0.05490452 0.03060114 0.0 rpy=3.14 0.0 0.0, axis 0 0 1, limit lower=-0.402 upper=0.402 effort=1000 velocity=2.0
- added joint robotiq_140_right_finger_joint: type fixed, parent robotiq_140_right_knuckle_link, child robotiq_140_right_finger_link, origin xyz=0.00795779 -0.03073656 0.0 rpy=0 0 0
- added joint robotiq_140_right_finger_tip_joint: type continuous, parent robotiq_140_right_inner_knuckle_link, child robotiq_140_right_finger_tip_link, origin xyz=0.09441861 -0.03294127  0.0 rpy=0.0 0.0 0.0, axis 0 0 1, limit lower=-3.14 upper=3.14 effort=0.1 velocity=100.0, mimic joint=robotiq_140_left_knuckle_joint multiplier=-1
- added joint robotiq_140_right_inner_knuckle_joint: type continuous, parent robotiq_140_base_link, child robotiq_140_right_inner_knuckle_link, origin xyz=0.06142 -0.0127 0 rpy=0 0 0, axis 0 0 1, limit lower=-3.14 upper=3.14 effort=0.1 velocity=100.0, mimic joint=robotiq_140_left_knuckle_joint offset=0
- added joint robotiq_140_right_knuckle_joint: type continuous, parent robotiq_140_base_link, child robotiq_140_right_knuckle_link, origin xyz=0.05490452 -0.03060114 0.0 rpy=0.0 0.0 0.0, axis 0 0 1, limit lower=-3.14 upper=3.14 effort=1000 velocity=100.0, mimic joint=robotiq_140_left_knuckle_joint

Commit message: fixed Joint_6 axis of rotation

File: src/fanuc/urdf/fanuc_gripper.urdf (robot description, URDF)
Before this commit: robot fanuc, 18 links, 17 joints
Joints:
- joint Joint_6: axis 0 0 0 -> 1 0 0

Commit message: joint limits updated

File: src/fanuc/urdf/fanuc_gripper.urdf (robot description, URDF)
Before this commit: robot fanuc, 18 links, 17 joints
Joints:
- joint Joint_1: limit lower=0 upper=6.632251 effort=0 velocity=2.094395 -> lower=-3.31613 upper=3.31613 effort=0 velocity=2.094395
- joint Joint_2: limit lower=0 upper=6.283185 effort=0 velocity=2.094395 -> lower=-3.14159 upper=3.14159 effort=0 velocity=2.094395
- joint Joint_3: limit lower=0 upper=9.948377 effort=0 velocity=3.141593 -> lower=-4.97419 upper=4.97419 effort=0 velocity=3.141593
- joint Joint_4: limit lower=0 upper=6.6323 effort=0 velocity=3.1416 -> lower=-3.31615 upper=3.31615 effort=0 velocity=3.1416
- joint Joint_5: limit lower=0 upper=6.2832 effort=0 velocity=3.1416 -> lower=-3.14159 upper=3.14159 effort=0 velocity=3.1416
- joint Joint_6: limit lower=0 upper=7.854 effort=0 velocity=3.1416 -> lower=-3.927 upper=3.927 effort=0 velocity=3.1416

Commit message: added inertia tensor tool and updated URDF inertia/mass values

File: src/fanuc/urdf/fanuc_gripper.urdf (robot description, URDF)
Before this commit: robot fanuc, 18 links, 17 joints
Links:
- link Link_1: mass 40 -> 3.84000000
- link Link_2: mass 40 -> 11.52000000
- link Link_3: mass 40 -> 2.88000000
- link Link_4: mass 40 -> 8.64000000
- link Link_5: mass 40 -> 1.60000000
- link Link_6: mass 40 -> 1.60000000
- link base_link: mass 40 -> 9.92000000

Commit message: eliminated unecessary info

File: src/fanuc/urdf/fanuc_gripper.urdf (robot description, URDF)
Before this commit: robot fanuc, 18 links, 17 joints
Links:
- removed link ee_link
Joints:
- removed joint ee_fixed_joint
- joint Joint_1: limit lower=-3.31613 upper=3.31613 effort=50 velocity=2.094395 -> lower=-3.31613 upper=3.31613 effort=330 velocity=2.094395
- joint Joint_2: limit lower=-3.14159 upper=3.14159 effort=45 velocity=2.094395 -> lower=-3.14159 upper=3.14159 effort=150 velocity=2.094395
- joint Joint_3: limit lower=-4.97419 upper=4.97419 effort=40 velocity=3.141593 -> lower=-4.97419 upper=4.97419 effort=55 velocity=3.141593
- joint robotiq_140_base_joint: parent ee_link -> Link_6
- joint robotiq_140_left_finger_tip_joint: limit lower=-3.14 upper=3.14 effort=0.1 velocity=100.0 -> (none)
- joint robotiq_140_left_inner_knuckle_joint: limit lower=-3.14 upper=3.14 effort=0.1 velocity=100.0 -> (none)
- joint robotiq_140_left_knuckle_joint: limit lower=-0.402 upper=0.402 effort=1000 velocity=2.0 -> lower=-0.3891 upper=0.3891 effort=1000 velocity=2.0
- joint robotiq_140_right_finger_tip_joint: limit lower=-3.14 upper=3.14 effort=0.1 velocity=100.0 -> (none)
- joint robotiq_140_right_inner_knuckle_joint: limit lower=-3.14 upper=3.14 effort=0.1 velocity=100.0 -> (none)
- joint robotiq_140_right_knuckle_joint: limit lower=-3.14 upper=3.14 effort=1000 velocity=100.0 -> (none)
